Commit message: chore: modified the robot to have steering wheels

File: src/dynamic_planner/urdf/my_bot.urdf (robot description, URDF)
Before this commit: robot simple_robot, 4 links, 3 joints
Joints:
- joint left_wheel_joint: origin xyz=0 -0.2 0.05 rpy=1.5708 0 0 -> xyz=0 -0.2 -0.1 rpy=1.5708 0 0
- joint right_wheel_joint: origin xyz=0 0.2 0.05 rpy=1.5708 0 0 -> xyz=0 0.2 -0.1 rpy=1.5708 0 0

Commit message: chore: added some files containing nav2

File: src/dynamic_planner/urdf/my_bot.urdf (robot description, URDF)
Before this commit: robot simple_robot, 4 links, 3 joints
Links:
- added link back_wheel, mass 0.2; collision cylinder length=0.05 radius=0.1; visual cylinder length=0.05 radius=0.1
- added link front_wheel, mass 0.2; collision cylinder length=0.05 radius=0.1; visual cylinder length=0.05 radius=0.1
Joints:
- added joint back_wheel_joint: type continuous, parent base_link, child back_wheel, origin xyz=-0.2 0 -0.1 rpy=1.5708 0 0, axis 0 0 1
- added joint front_wheel_joint: type continuous, parent base_link, child front_wheel, origin xyz=0.2 0 -0.1 rpy=1.5708 0 0, axis 0 0 1
